Commit message: add imu

File: custom_husky/urdf/custom_husky.urdf (robot description, URDF)
Before this commit: robot custom_husky, 10 links, 9 joints
Links:
- added link imu_link, mass 0.01; collision box size=0.02 0.02 0.01; visual box size=0.02 0.02 0.01
Joints:
- added joint imu_joint: type fixed, parent base_link, child imu_link, origin xyz=0 0 1 rpy=0 0 0

File: custom_husky/urdf/custom_husky.urdf.xacro (robot description, xacro)
@@ -316,9 +316,46 @@
         <child link="camera"/>
     </joint>
-    <!-- ROS2 Control Plugin -->
-    <gazebo>
-      <plugin name="gazebo_ros2_control" filename="libgazebo_ros2_control.so">
-        <!-- <parameters>$(arg gazebo_controllers)</parameters> -->
-      </plugin>
+    <link name="imu_link">
+        <visual>
+            <origin xyz="0 0 0" rpy="0 0 0"/>
+            <geometry>
+                <box size="0.02 0.02 0.01"/>
+            </geometry>
+            <material name="red"/>
+        </visual>
+        <collision>
+            <origin xyz="0 0 0" rpy="0 0 0"/>
+            <geometry>
+                <box size="0.02 0.02 0.01"/>
+            </geometry>
+        </collision>
+        <inertial>
+            <origin xyz="0 0 0" rpy="0 0 0"/>
+            <mass value="0.01"/>
+            <inertia ixx="1e-6" ixy="0.0" ixz="0.0"
+                     iyy="1e-6" iyz="0.0"
+                     izz="1e-6"/>
+        </inertial>
+    </link>
+    <joint name="imu_joint" type="fixed">
+        <origin xyz="0 0 1" rpy="0 0 0"/>
+        <parent link="base_link"/>
+        <child link="imu_link"/>
+    </joint>
+    <gazebo reference="imu_link">
+        <sensor type="imu" name="imu_sensor">
+        <always_on>true</always_on>
+        <update_rate>50</update_rate>
+        <visualize>true</visualize>
+        <plugin name="imu_plugin" filename="libgazebo_ros_imu_sensor.so">
+            <ros>
+                <namespace>/</namespace>
+                <remapping>imu_plugin/out:=imu/data</remapping>
+            </ros>
+        <body_name>imu_link</body_name>
+        <frame_name>imu_link</frame_name>
+        <gaussian_noise>0.01</gaussian_noise>
+        </plugin>
+        </sensor>
     </gazebo>
 </robot>

Commit message: update imu_link

File: custom_husky/urdf/custom_husky.urdf (robot description, URDF)
Before this commit: robot custom_husky, 11 links, 10 joints
Links:
- link imu_link: mass 0.01 -> None; geometry 
Joints:
- joint imu_joint: origin xyz=0 0 1 rpy=0 0 0 -> xyz=0 0 0 rpy=0 0 0

File: custom_husky/urdf/custom_husky.urdf.xacro (robot description, xacro)
@@ -316,28 +316,8 @@
         <child link="camera"/>
     </joint>
-    <link name="imu_link">
-        <visual>
-            <origin xyz="0 0 0" rpy="0 0 0"/>
-            <geometry>
-                <box size="0.02 0.02 0.01"/>
-            </geometry>
-            <material name="red"/>
-        </visual>
-        <collision>
-            <origin xyz="0 0 0" rpy="0 0 0"/>
-            <geometry>
-                <box size="0.02 0.02 0.01"/>
-            </geometry>
-        </collision>
-        <inertial>
-            <origin xyz="0 0 0" rpy="0 0 0"/>
-            <mass value="0.01"/>
-            <inertia ixx="1e-6" ixy="0.0" ixz="0.0"
-                     iyy="1e-6" iyz="0.0"
-                     izz="1e-6"/>
-        </inertial>
-    </link>
+    <!-- IMU Link -->
+    <link name="imu_link"/>
     <joint name="imu_joint" type="fixed">
-        <origin xyz="0 0 1" rpy="0 0 0"/>
+        <origin xyz="0 0 0" rpy="0 0 0"/>
         <parent link="base_link"/>
         <child link="imu_link"/>

Commit message: fix camera frame

File: custom_husky/urdf/custom_husky.urdf (robot description, URDF)
Before this commit: robot custom_husky, 11 links, 10 joints
Links:
- added link camera_optical_link
Joints:
- added joint camera_optical_joint: type fixed, parent camera, child camera_optical_link, origin xyz=0 0 0 rpy=-1.5708 0 -1.5708

File: custom_husky/urdf/custom_husky.urdf.xacro (robot description, xacro)
@@ -322,4 +322,11 @@
         <child link="camera_mount"/>
     </joint>
+    <!-- Camera Optical Link -->
+    <link name="camera_optical_link"/>
+    <joint name="camera_optical_joint" type="fixed">
+        <origin xyz="0 0 0" rpy="-1.5708 0 -1.5708"/>
+        <parent link="camera"/>
+        <child link="camera_optical_link"/>
+    </joint>
     <!-- Camera -->
     <link name="camera">
@@ -366,5 +373,5 @@
             <plugin name="depth_camera_driver" filename="libgazebo_ros_camera.so">
                 <cameraName>depth_camera</cameraName>
-                <frameName>camera</frameName>
+                <frameName>camera_optical_link</frameName>
                 <imageTopicName>image_raw</imageTopicName>
                 <cameraInfoTopicName>depth/camera_info</cameraInfoTopicName>

Commit message: tune rpy camera_optical_link

File: custom_husky/urdf/custom_husky.urdf (robot description, URDF)
Before this commit: robot custom_husky, 12 links, 11 joints
Joints:
- joint camera_optical_joint: origin xyz=0 0 0 rpy=-1.5708 0 -1.5708 -> xyz=0 0 0 rpy=0 -1.5708 1.5708

File: custom_husky/urdf/custom_husky.urdf.xacro (robot description, xacro)
@@ -325,5 +325,5 @@
     <link name="camera_optical_link"/>
     <joint name="camera_optical_joint" type="fixed">
-        <origin xyz="0 0 0" rpy="-1.5708 0 -1.5708"/>
+        <origin xyz="0 0 0" rpy="0 -1.5708 1.5708"/>
         <parent link="camera"/>
         <child link="camera_optical_link"/>

Commit message: fix camera frame issue

File: custom_husky/urdf/custom_husky.urdf (robot description, URDF)
Before this commit: robot custom_husky, 12 links, 11 joints
Joints:
- joint camera_optical_joint: origin xyz=0 0 0 rpy=0 -1.5708 1.5708 -> xyz=0 0 0 rpy=-1.5707963267948966 0 -1.5707963267948966

File: custom_husky/urdf/custom_husky.urdf.xacro (robot description, xacro)
@@ -325,5 +325,5 @@
     <link name="camera_optical_link"/>
     <joint name="camera_optical_joint" type="fixed">
-        <origin xyz="0 0 0" rpy="0 -1.5708 1.5708"/>
+        <origin xyz="0 0 0" rpy="-${pi/2} 0 -${pi/2}"/>
         <parent link="camera"/>
         <child link="camera_optical_link"/>
@@ -360,5 +360,5 @@
             <pose>0 0 0 0 0 0</pose>
             <depth_camera name="depth_cam">
-                <horizontal_fov>1.3962634</horizontal_fov> <!-- ~80 degrees -->
+                <horizontal_fov>2</horizontal_fov>
                 <image>
                     <width>320</width>
@@ -372,13 +372,5 @@
             </depth_camera>
             <plugin name="depth_camera_driver" filename="libgazebo_ros_camera.so">
-                <cameraName>depth_camera</cameraName>
-                <frameName>camera_optical_link</frameName>
-                <imageTopicName>image_raw</imageTopicName>
-                <cameraInfoTopicName>depth/camera_info</cameraInfoTopicName>
-                <depthImageTopicName>depth/image_raw</depthImageTopicName>
-                <depthImageCameraInfoTopicName>depth/camera_info</depthImageCameraInfoTopicName>
-                <pointCloudTopicName>depth/points</pointCloudTopicName>
-                <outputDepthImage>true</outputDepthImage>
-                <outputPointCloud>true</outputPointCloud>
+                <frame_name>camera_optical_link</frame_name>
             </plugin>
         </sensor>
